Commit message: Update 30m road and lidar geometry

File: src/avoidance_gazebo/urdf/turtle_car.urdf.xacro (robot description, xacro)
@@ -24,10 +24,9 @@
   <xacro:property name="steering_link_radius" value="0.020"/>
   <xacro:property name="steering_link_height" value="0.040"/>
-  <!-- Low under the front body, inside the bumper and below the chassis
-       collision, whose lower face remains at z=0.15. -->
-  <xacro:property name="laser_x" value="0.55"/>
+  <!-- LiDAR centres are on the vehicle front/rear end planes. -->
+  <xacro:property name="laser_x" value="0.65"/>
   <xacro:property name="laser_z_from_ground" value="0.12"/>
-  <xacro:property name="laser_radius" value="0.025"/>
-  <xacro:property name="laser_height" value="0.040"/>
+  <xacro:property name="laser_radius" value="0.050"/>
+  <xacro:property name="laser_height" value="0.080"/>
   <!-- Total model mass is approximately 21.05 kg. -->
   <xacro:property name="chassis_mass" value="18.0"/>
@@ -221,4 +220,9 @@
       <material name="laser_black"/>
     </visual>
+    <collision>
+      <geometry>
+        <cylinder radius="${laser_radius}" length="${laser_height}"/>
+      </geometry>
+    </collision>
   </link>
   <joint name="laser_joint" type="fixed">
@@ -240,4 +244,9 @@
       <material name="laser_black"/>
     </visual>
+    <collision>
+      <geometry>
+        <cylinder radius="${laser_radius}" length="${laser_height}"/>
+      </geometry>
+    </collision>
   </link>
   <joint name="rear_laser_joint" type="fixed">
